Commit message: Retificação do LIDAR e voxblox planner
O LIDAR só lê para a frente
Voxblox planner ainda não está a funcionar totalmente

Signed-off-by: protobella <marianaleucadio@gmail.com>

File: sjtu-drone/urdf/velodyne.xacro (robot description, xacro)
@@ -2,5 +2,5 @@
 <robot xmlns:xacro="http://www.ros.org/wiki/xacro" name="HDL-32E">
   <xacro:property name="M_PI" value="3.1415926535897931" />
-  <xacro:macro name="HDL-32E" params="*origin parent:=base_link name:=velodyne topic:=/velodyne_points organize_cloud:=false hz:=10 lasers:=32 samples:=2187 collision_range:=0.3 min_range:=0.9 max_range:=130.0 noise:=0.008 min_angle:=-${M_PI} max_angle:=${M_PI} gpu:=false">
+  <xacro:macro name="HDL-32E" params="*origin parent:=base_link name:=velodyne topic:=/velodyne_points organize_cloud:=false hz:=10 lasers:=32 samples:=32 collision_range:=0.05 min_range:=0.9 max_range:=69.0 noise:=0.008 min_angle:=-0.53529248 max_angle:=0.53529248 gpu:=false">
     <joint name="${name}_base_mount_joint" type="fixed">
       <xacro:insert_block name="origin" />
@@ -76,5 +76,5 @@
               <min>${collision_range}</min>
               <max>${max_range+1}</max>
-              <resolution>0.001</resolution>
+              <resolution>0.02</resolution>
             </range>
             <noise>
@@ -97,5 +97,5 @@
         <sensor type="ray" name="${name}-HDL32E">
           <pose>0 0 0 0 0 0</pose>
-          <visualize>false</visualize>
+          <visualize>true</visualize>
           <update_rate>${hz}</update_rate>
           <ray>

Commit message: Implementação da voxblox mesh e o LiDAR faz o scan só para a frente
Signed-off-by: protobella <marianaleucadio@gmail.com>

File: sjtu-drone/urdf/velodyne.xacro (robot description, xacro)
@@ -2,5 +2,5 @@
 <robot xmlns:xacro="http://www.ros.org/wiki/xacro" name="HDL-32E">
   <xacro:property name="M_PI" value="3.1415926535897931" />
-  <xacro:macro name="HDL-32E" params="*origin parent:=base_link name:=velodyne topic:=/velodyne_points organize_cloud:=false hz:=10 lasers:=32 samples:=2187 collision_range:=0.3 min_range:=0.9 max_range:=130.0 noise:=0.008 min_angle:=-${M_PI} max_angle:=${M_PI} gpu:=false">
+  <xacro:macro name="HDL-32E" params="*origin parent:=base_link name:=velodyne topic:=/velodyne_points organize_cloud:=false hz:=10 lasers:=32 samples:=32 collision_range:=0.05 min_range:=0.9 max_range:=69.0 noise:=0.008 min_angle:=-0.53529248 max_angle:=0.53529248 gpu:=false">
     <joint name="${name}_base_mount_joint" type="fixed">
       <xacro:insert_block name="origin" />
