Commit message: Implementação de waypoints a volta dos carros
Signed-off-by: protobella <marianaleucadio@gmail.com>

File: sjtu-drone/urdf/sjtu_drone.urdf.xacro (robot description, xacro)
@@ -55,5 +55,5 @@
   <!-- Sensors -->
   <gazebo reference="base_link">
-    	<!-- <sensor name='sensor_imu' type='imu'>
+    	<sensor name='sensor_imu' type='imu'>
         <always_on> 1 </always_on>
         <update_rate> 100 </update_rate>
@@ -74,5 +74,5 @@
           </noise>
         </imu>
-      </sensor> -->
+      </sensor>
       <!-- Sonar sensor in 100fps -->
       <!-- <sensor name='sensor_sonar' type='sonar'>

File: sjtu-drone/urdf/velodyne.xacro (robot description, xacro)
@@ -2,5 +2,5 @@
 <robot xmlns:xacro="http://www.ros.org/wiki/xacro" name="HDL-32E">
   <xacro:property name="M_PI" value="3.1415926535897931" />
-  <xacro:macro name="HDL-32E" params="*origin parent:=base_link name:=velodyne topic:=/velodyne_points organize_cloud:=false hz:=10 lasers:=32 samples:=32 collision_range:=0.05 min_range:=0.9 max_range:=69.0 noise:=0.008 min_angle:=-0.53529248 max_angle:=0.53529248 gpu:=false">
+  <xacro:macro name="HDL-32E" params="*origin parent:=base_link name:=velodyne topic:=/velodyne_points organize_cloud:=false hz:=10 lasers:=32 samples:=2187 collision_range:=0.3 min_range:=0.9 max_range:=130.0 noise:=0.008 min_angle:=-${M_PI} max_angle:=${M_PI} gpu:=false">
     <joint name="${name}_base_mount_joint" type="fixed">
       <xacro:insert_block name="origin" />
